File: CartridgeTemplate.kicad_pcb (KiCad board)
At the start: 2 copper layers, 64.8 x 55.9 mm, 3 parts, among them J1 Cartridge Connector, U1 W25Q128

Commit message: Added badge outline in Dwgs.Use
This is not the exact outline, but a guess based on the official proto breakout cartridge and a photo of a badge
Other:
- net class Default: clearance 0.1524 -> 0.2; trace_width 0.1524 -> 0.25
- rule trace_clearance: 0.1524 -> 0.2
- rule trace_min: 0.1524 -> 0.2
Changed lines of the file:
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@@
   (general
     (thickness 1.6)
-    (drawings 59)
+    (drawings 74)
     (tracks 36)
     (zones 0)
@@
   )
   (setup
-    (last_trace_width 0.2032)
+    (last_trace_width 0.25)
     (user_trace_width 0.2032)
     (user_trace_width 0.254)
     (user_trace_width 0.3048)
-    (trace_clearance 0.1524)
-    (zone_clearance 0.1524)
+    (trace_clearance 0.2)
+    (zone_clearance 0.508)
     (zone_45_only no)
-    (trace_min 0.1524)
+    (trace_min 0.2)
     (via_size 0.8)
     (via_drill 0.4)
@@
     (pcb_text_width 0.3)
     (pcb_text_size 1.5 1.5)
-    (mod_edge_width 0.12)
+    (mod_edge_width 0.3)
     (mod_text_size 1 1)
     (mod_text_width 0.15)
@@
     (pad_to_mask_clearance 0.051)
     (solder_mask_min_width 0.25)
-    (aux_axis_origin 67.31 50.8)
+    (aux_axis_origin 102 84)
     (grid_origin 101.6 50.8)
     (visible_elements FFFFFF7F)
     (pcbplotparams
-      (layerselection 0x010fc_ffffffff)
+      (layerselection 0x210a8_7fffffff)
       (usegerberextensions false)
       (usegerberattributes false)
@@
       (creategerberjobfile false)
       (excludeedgelayer true)
-      (linewidth 0.050000)
+      (linewidth 0.100000)
       (plotframeref false)
       (viasonmask false)
@@
       (padsonsilk false)
       (subtractmaskfromsilk false)
-      (outputformat 1)
+      (outputformat 4)
       (mirror false)
-      (drillshape 1)
+      (drillshape 0)
       (scaleselection 1)
-      (outputdirectory ""))
+      (outputdirectory "prod/"))
   )
   (net 0 "")
@@
   (net 40 +BATT)
   (net_class Default "This is the default net class."
-    (clearance 0.1524)
-    (trace_width 0.1524)
+    (clearance 0.2)
+    (trace_width 0.25)
     (via_dia 0.8)
     (via_drill 0.4)
@@
     )
   )
+  (gr_circle (center 64.45 47.425) (end 67.95 47.425) (layer Dwgs.User) (width 0.15))
+  (gr_line (start 50.075 85.55) (end 50.075 105.525) (layer Dwgs.User) (width 0.15))
+  (gr_line (start 53.575 82.05) (end 50.075 85.55) (layer Dwgs.User) (width 0.15))
+  (gr_line (start 53.575 47.4) (end 53.575 82.05) (layer Dwgs.User) (width 0.15))
+  (gr_line (start 59.575 41.4) (end 53.575 47.4) (layer Dwgs.User) (width 0.15))
+  (gr_line (start 69.55 41.4) (end 59.575 41.4) (layer Dwgs.User) (width 0.15))
+  (gr_line (start 75.775 47.4) (end 69.55 41.4) (layer Dwgs.User) (width 0.15))
   (gr_arc (start 62.228261 60.957825) (end 68.578261 66.037824) (angle -77.3) (layer B.SilkS) (width 1))
   (gr_arc (start 137.16 60.96) (end 130.810001 55.880001) (angle -77.3) (layer B.SilkS) (width 1))
@@
   (gr_line (start 76.2 106.68) (end 127 106.68) (layer Edge.Cuts) (width 0.05))
   (gr_line (start 101.6 25.4) (end 101.6 177.8) (layer Dwgs.User) (width 0.15))
+  (gr_line (start 135.375 54.1) (end 135.375 100.7) (layer Dwgs.User) (width 0.15))
+  (gr_line (start 135.375 51.1) (end 135.175 50.9) (layer Dwgs.User) (width 0.15))
+  (gr_line (start 135.375 54.1) (end 135.375 51.1) (layer Dwgs.User) (width 0.15))
+  (gr_line (start 135.375 100.7) (end 135.375 105.5) (layer Dwgs.User) (width 0.15))
+  (gr_line (start 135.175 50.9) (end 128.175 43.9) (layer Dwgs.User) (width 0.15))
+  (gr_line (start 86.775 43.9) (end 128.175 43.9) (layer Dwgs.User) (width 0.15))
+  (gr_line (start 83.275 47.4) (end 86.775 43.9) (layer Dwgs.User) (width 0.15))
+  (gr_line (start 75.775 47.4) (end 83.275 47.4) (layer Dwgs.User) (width 0.15))
   (segment (start 75.565 88.265) (end 72.5 88.265) (width 0.1524) (layer F.Cu) (net 2))
   (segment (start 77.47 90.17) (end 75.565 88.265) (width 0.1524) (layer F.Cu) (net 2))
